File: LED Driver.brd (EAGLE design)
At the start: 21.3 x 25.4 mm, 10 parts, among them IC1 LM4041A12DBZ

Commit message: Fixed board asthetics
Added labels for input terminals, fixed logo, changed text to Revision B
Parts:
- R2: value 90k -> 240k
Other:
- board text added: "+"
- board text added: "-"
- board text added: "DIM"
- board text added: "LED"
- board text added: "PWR"
- board text added: "Revision B"
- board text removed: "Revision A"
